File: dropper_torpedo/dropper_torpedo.sch (EAGLE design)
At the start: 15 parts, among them Q1 IRFZ48Z, Q2 IRFZ48Z, T1 BD139, T2 BD139

Commit message: Complete dropper torpedo board
Parts:
- removed D1, D2: 1N4004, diode:1N4004
- removed JP5: (no value), adafruit:PINHD-1X3
- removed Q1, Q2: IRFZ48Z, transistor-power:IRFZ48Z
- removed T1, T2: BD139, transistor:BD139
- added D24V22F5: (no value), SparkFun:M05PTH
- added D3, D4: 1N4004, diode:1N4004
- added INPUT: (no value), SparkFun:M04POLAR
- added LED1, LED2, LED3: (no value), SparkFun:LED0603
- added Q3, Q4: IRFZ48Z, transistor-power:IRFZ48Z
- added R4: 560R, SparkFun:RESISTOR0805-RES
- added R5, R6, R7: 10K, SparkFun:RESISTOR0805-RES
- added SERVO_L, SERVO_R, TORPEDO_L, TORPEDO_R: (no value), SparkFun:M03POLAR
- added T3, T4: BD139, transistor:BD139
- added U$1: ARVP_LOGO, ARVP:ARVP_LOGO
- JP1: value (none) -> STAND-OFF; device adafruit:PINHD-1X6 -> SparkFun:STAND-OFF
- JP2, JP3, JP4: value (none) -> STAND-OFF; device adafruit:PINHD-1X3 -> SparkFun:STAND-OFF
- R1, R2: value 10 K -> 150R; device adafruit:R-US_0204/7 -> SparkFun:RESISTOR0805-RES
- R3: value 10 K -> 10K; device adafruit:R-US_0204/7 -> SparkFun:RESISTOR0805-RES
Connections:
- removed net 12V: D1.C, D2.C, JP1.4, JP4.2, JP5.2, U$2.9V
- removed net 5V: JP1.3, T1.C
- removed net N$11: T2.E
- removed net N$2: Q1.G, R2.1, U$2.8
- removed net N$6: D1.A, JP4.3, Q2.D
- removed net N$7: JP3.2, T1.E
- removed net N$8: D2.A, JP5.3, Q1.D
- removed net N$9: T2.B, U$2.10
- new net +12V: D24V22F5.3, D3.C, D4.C, INPUT.1, LED1.A, TORPEDO_L.2, TORPEDO_R.2, U$2.9V
- new net +5V: D24V22F5.1, T3.C, T4.C
- new net N$10: LED1.C, R4.2
- new net N$13: SERVO_L.2, T3.E
- new net N$14: SERVO_R.2, T4.E
- new net S_ENL: R5.2, T3.B, U$2.7
- new net S_ENR: R6.2, T4.B, U$2.8
- new net S_SIGL: SERVO_L.1, U$2.5
- new net S_SIGR: SERVO_R.1, U$2.6
- new net TOR_L: LED2.A, Q3.G, R3.2, U$2.9
- new net TOR_R: LED3.A, Q4.G, R7.2, U$2.10
- net GND: now also D24V22F5.2, INPUT.4, Q3.S, Q4.S, R1.1, R2.1, R3.1, R4.1, R5.1, R6.1, R7.1, SERVO_L.3, SERVO_R.3, U$2.GND@1; no longer JP1.1, JP2.3, JP3.3, Q1.S, Q2.S, R1.2, R2.2, R3.2
- net N$1: now also D3.A, Q3.D, TORPEDO_L.1; no longer R3.1, T1.B, U$2.7
- net N$3: now also LED2.C, R1.2; no longer Q2.G, R1.1, U$2.9
- net N$4: now also D4.A, Q4.D, TORPEDO_R.1; no longer JP3.1, U$2.6
- net N$5: now also LED3.C, R2.2; no longer JP2.1, U$2.5
- net RX: now also INPUT.2; no longer JP1.5
- net TX: now also INPUT.3; no longer JP1.6
Other:
- note added: "1.0"
- note added: "Eric Wells"
- note added: "Rumman Waqar"
- moved on the sheet: R1, R2, R3
